File: temp_reg.sch (KiCad schematic (older format))
At the start: 125 parts

Commit message: milestone version
Parts:
- removed 100uF, 100uF? (x2), C? (x2): CP, symbol CP
- removed 330R, 330R? (x2), R? (x12): R, symbol R
- removed C?: CP1_Small, symbol CP1_Small
- removed C? (x5): C_Small, symbol C_Small
- removed JP? (x3): Jumper_NO_Small, symbol Jumper_NO_Small
- removed R? (x3): 1k, symbol R
- removed RV?: POT, symbol POT
- removed U? (x2): MCP3201-CI/SN, SOIC127P600X175-8N, symbol MCP3201-CI/SN-RESCUE-temp_reg-RESCUE-temp_reg
- removed U? (x3): TL082, symbol TL082
- added 100n (x3), 100n? (x4), 10n, C? (x6): C_Small, symbol C_Small
- added 100u (x2), 4.7u (x2), 4.7u? (x3), 47u (x2), C? (x3): CP1_Small, symbol CP1_Small
- added 100uF? (x3): CP, symbol CP
- added 1R, 330R? (x6), R? (x9): R, symbol R
- added JP? (x3): Jumper_NO_Small, symbol Jumper_NO_Small
- added P?: CONN_01X04, symbol CONN_01X04
- added P? (x6): CONN_01X01, symbol CONN_01X01
- added U? (x3): MCP3201-CI/SN, SOIC127P600X175-8N, symbol MCP3201-CI/SN-RESCUE-temp_reg-RESCUE-temp_reg
- added U? (x3): TL082, symbol TL082
- added U?: LM7805, symbol LM7805
- added W? (x6): TEST_1P, symbol TEST_1P
- U?: symbol LM337T -> LM337T-RESCUE-temp_reg
- gave numbers to parts that had none: 12
Connections:
- net labels added: CS_ADC2, RST, VCC, ctl, mes_A, mes_B, mes_C
- net labels removed: DAC_A
- wire segments 435 -> 393
Other:
- note added: "on / off"
- note added: "on/off wire heating"
- note added: "prog"
- note removed: "on/off wire"
- moved on the sheet: 100n, 100u, 10k, 10u, 1R, 20MHz, 220R, 22p, 30k, 330R, 47u, 560R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

Commit message: boost converter version
Parts:
- removed 100n (x6), 100n? (x3), 10n, C? (x4): C_Small, symbol C_Small
- removed 100u (x3), 10u, 4.7u (x2), 4.7u? (x2), 47u: CP1_Small, symbol CP1_Small
- removed 100uF? (x3), C? (x3): CP, symbol CP
- removed 10k (x2), 1R (x2), 30k, 330R, 330R? (x6), 560R, R? (x8): R, symbol R
- removed C? (x2): C, symbol C
- removed D? (x2): D, symbol D
- removed D?: Led_Small, symbol Led_Small
- removed P?: CONN_2vert, symbol CONN_2vert
- removed Q?: Q_NPN_EBC, symbol Q_NPN_EBC
- removed U?: LM337T, TO-220, symbol LM337T-RESCUE-temp_reg
- removed U?: MCP4822-s, SOP65P490X110-8N, symbol MCP4822-s-RESCUE-temp_reg
- removed U? (x4): TL082, symbol TL082
- removed U? (x2): MCP3201-CI/SN, SOIC127P600X175-8N, symbol MCP3201-CI/SN-RESCUE-temp_reg-RESCUE-temp_reg
- removed W? (x6): TEST_1P, symbol TEST_1P
- added 100n, 100n? (x7): C_Small, symbol C_Small
- added 1R? (x2), R? (x18): R, symbol R
- added 4.7u? (x3), 47u? (x2): CP1_Small, symbol CP1_Small
- added C? (x2): CP, symbol CP
- added D? (x2): D_Schottky_Small, symbol D_Schottky_Small
- added L? (x5): L, symbol L
- added P?: CONN_2vert, symbol CONN_2vert
- added P?: CONN_01X04, symbol CONN_01X04
- added P? (x2): CONN_01X02, symbol CONN_01X02
- added Q? (x2): Q_NMOS_DSG, symbol Q_NMOS_DSG
- added RV?: POT, symbol POT
- added U? (x2): MCP601P, Housings_DIP:DIP-8_W7.62mm, symbol MCP601P
- added U? (x2): LM393, symbol LM393
- added U?: MCP3201-CI/SN, SOIC127P600X175-8N, symbol MCP3201-CI/SN-RESCUE-temp_reg-RESCUE-temp_reg
- RV? (x2): symbol POT -> POT-RESCUE-temp_reg
- renumbered 47u to 10u
Connections:
- net CS_ADC2 is gone; now on net CS_ADC_B: U?.5 (~CS/SHDN)
- net CS_DAC1 is gone; now on net D7: IC?.3 ((PCINT10/AIN0/INT2)PB2)
- net +12V: now also 47u?.1, D?.2 (A), L?.2, L?.2; no longer 100n.1, 10u.1, U?.VI
- net +5V: now also RV?.3; no longer 100n.1, 100n?.1, 10k.2, 4.7u?.1, 47u.1, 47u.1, R?.2, RV?.1, U?.8 (VDD), U?.VO
- net BEEP: now also IC?.37 ((PCINT3/ADC3)PA3); no longer IC?.20 ((PCINT30/OC2B/ICP)PD6)
- net D6: now also IC?.22 ((PCINT16/SCL)PC0); no longer IC?.15 ((PCINT25/TXD0)PD1)
- net D7: no longer IC?.14 ((PCINT24/RXD0)PD0)
- net ESTOP: now also P?.1 (P1)
- net GND: now also RV?.3, 100n.2, 100n?.2, 100n?.2, 47u?.2, C?.2, C?.2, L?.2, R?.1, R?.1, R?.1, U?.4 (V-), U?.4 (V-); no longer 100n.2, 100n.2, 100n?.2, 10u.2, 4.7u?.2, 47u.2, 47u.2, 47u.2, D?.2 (A), RV?.2, U?.3 (IN-), U?.4 (VSS), U?.GND
- net JP_1: now also P?.4 (P4)
- net JP_2: now also P?.3 (P3)
- net JP_3: now also P?.2 (P2)
- net LED_1: now also IC?.21 ((PCINT31/OC2A)PD7)
- net LED_2: now also IC?.20 ((PCINT30/OC2B/ICP)PD6)
- net MOSI: now also U?.6 (DOUT)
- net SCK: now also U?.7 (CLK)
- net VCC: now also 10k.2, RV?.1
- net Vref: now also RV?.3, U?.1 (VREF); no longer D?.3 (Ref)
- net mes_B: now also 1R?.2, P?.2 (P2), R?.2
- net at DS?.3 (VO): now also RV?.2; no longer RV?.1
- net at C?.1, R?.2, U?.2 (TRIG)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: now also RV?.1
- net PWM: now reaches IC?.1 ((PCINT8/T0/XCK)PB0)
- net PWM: now also U?.3 (+)
- net at IC?.32 (AREF): now also 100n.1
- net CS_ADC_B: now reaches IC?.4 ((PCINT11/AIN1/OC0A)PB3)
- net CS_ADC_A: now reaches IC?.5 ((PCINT12/OC0B/SS)PB4)
- net CS_ADC_A: now also U?.5 (~CS/SHDN)
- net at U?.2 (IN+): now also 100n?.1, R?.1, U?.6
- net DAC1_L renamed PWM_ON/OFF
- net PWM_ON/OFF: now also U?.5 (+)
- new net: 100n.1, 10u.1, 47u?.1, L?.1, U?.VI
- new net: D?.3 (Ref), RV?.2
- new net: 47u.1, L?.1, R?.2
- new net: IC?.14 ((PCINT24/RXD0)PD0), P?.1 (P1)
- new net: IC?.15 ((PCINT25/TXD0)PD1), P?.2 (P2)
- new net: R?.1, R?.2, R?.2 (x2)
- new net: R?.2, R?.2, U?.2 (-) (x2)
- new net: 100n?.1, R?.1, U?.3 (+) (x2)
- new net: 100n?.2, R?.1, R?.2 (x2)
- new net: 100n?.1, R?.1, U?.2 (IN+), U?.6
- new net: 1R?.1, 4.7u?.1, D?.1 (K)
- new net: L?.1, Q?.2 (S)
- new net: D?.2 (A), L?.2, Q?.1 (D)
- new net: Q?.3 (G), R?.1, R?.2
- new net: R?.1, U?.1
- new net: R?.1, R?.2, U?.2 (_), U?.6 (_)
- new net: 100n?.1, C?.1, L?.1, R?.2, R?.2, R?.2, U?.8 (V+), U?.8 (V+)
- new net: 100n?.1, C?.1, D?.1 (K), Q?.1 (D)
- new net: Q?.3 (G), R?.1, R?.1
- new net: R?.2, U?.7
- new net AVCC: 100n.1, 100n?.1, 100n?.1, 4.7u?.1, 4.7u?.1, 47u.1, L?.2, P?.2 (P2), U?.7 (V+), U?.7 (V+), U?.8 (VDD), U?.8 (VDD), U?.VO
- new net GNDA: 100n.2, 100n.2, 100n?.2, 100n?.2, 100n?.2, 100n?.2, 10u.2, 4.7u?.2, 4.7u?.2, 47u.2, 47u.2, 47u.2, 47u?.2, D?.2 (A), L?.1, P?.1 (P1), R?.1, R?.1, RV?.1, U?.3 (IN-), U?.3 (IN-), U?.4 (V-), U?.4 (V-), U?.4 (VSS), U?.4 (VSS), U?.GND
- new net GNDPWR: 4.7u?.2, 4.7u?.2, P?.1 (P1), Q?.2 (S)
- new net mes_A: 1R?.1, 1R?.2, 4.7u?.1, R?.2
Other:
- moved on the sheet: 100n, 100n?, 10k, 20MHz, 22p, 4.7u?, 47u, C?, D?, IC?, P?, Q?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
