File: temp_reg.sch (KiCad schematic (older format))
At the start: 133 parts, among them IC1 ATMEGA644-P, P1 CONN_01X02, P10 CONN_01X04, P11 CONN_01X06, P12 CONN_01X02, P13 CONN_01X02, P15 CONN_01X02, P2 CONN_01X03, P3 CONN_01X03, P4 CONN_2, P5 CONN_01X02, P6 CONN_01X04, P7 CONN_01X06, P8 CONN_01X05, P9 CONN_01X01, U10 LM7805, U11 LM7805, U5 EL817C, U7 EL817C, U8 EL817C, U9 EL817C

Commit message: change to modular architecture
Parts:
- removed 100n5, 22p1, 22p2, C7, C8: C_Small, Capacitors_THT:C_Disc_D3.0mm_W1.6mm_P2.50mm, symbol C_Small
- removed 20MHz1: Crystal, Crystals:Resonator-2pin_w7.0mm_h2.5mm, symbol Crystal
- removed 220R3, R17, R19, R21, R31, R32: R, Resistors_THT:Resistor_Horizontal_RM7mm, symbol R
- removed 47u1, 47u4, 47u5, 47u6, 47u?: CP1_Small, Capacitors_THT:CP_Radial_D4.0mm_P1.50mm, symbol CP1_Small
- removed C5, C6, C9: CP1_Small, Capacitors_THT:C_Radial_D5_L6_P2.5, symbol CP1_Small
- removed D1, D2: Led_Small, LEDs:LED_D3.0mm, symbol Led_Small
- removed D5: TL431, TO_SOT_Packages_THT:TO-92_Inline_Narrow_Oval, symbol TL431
- removed D? (x5): LED, symbol LED
- removed IC1: ATMEGA644-P, Housings_DIP:DIP-40_W25.4mm_Socket_LongPads, symbol ATMEGA644-P
- removed JP1, JP2, JP3, JP4: Jumper_NO_Small, Buttons_Switches_THT:SW_PUSH_6mm_h4.3mm, symbol Jumper_NO_Small
- removed L3, L4, L5, L6, L7: L, Resistors_THT:Resistor_Horizontal_RM7mm, symbol L
- removed P1, P13: CONN_01X02, Pin_Headers:Pin_Header_Straight_1x02_Pitch2.54mm, symbol CONN_01X02
- removed P10: CONN_01X04, Pin_Headers:Pin_Header_Straight_1x04_Pitch2.54mm, symbol CONN_01X04
- removed P11, P7: CONN_01X06, Pin_Headers:Pin_Header_Straight_1x06_Pitch2.54mm, symbol CONN_01X06
- removed P3: CONN_01X03, Pin_Headers:Pin_Header_Straight_1x03_Pitch2.54mm, symbol CONN_01X03
- removed P8: CONN_01X05, Pin_Headers:Pin_Header_Straight_1x05_Pitch2.54mm, symbol CONN_01X05
- removed P?: CONN_01X02, symbol CONN_01X02
- removed Q? (x4): Q_NPN_CBE, symbol Q_NPN_CBE
- removed R? (x20): R, symbol R
- removed RV1: POT, Potentiometers:Potentiometer_Trimmer_Bourns_3296W, symbol POT
- removed RV2: POT, Potentiometers:Potentiometer_Trimmer_Bourns_3296W, symbol POT-RESCUE-temp_reg
- removed S? (x3): 7SEGM, symbol 7SEGM
- removed U10: LM7805, TO_SOT_Packages_THT:TO-220_Vertical, symbol LM7805-RESCUE-temp_reg
- removed U8: EL817C, Housings_DIP:DIP-4_W7.62mm, symbol EL817C-RESCUE-temp_reg
- removed U?: MCP601P, Housings_DIP:DIP-8_W7.62mm, symbol MCP601P
- removed U? (x2): 74HC595, symbol 74HC595
- removed U?: 7400, symbol 7400
- added C? (x3): CP, symbol CP
- added D?: TL431, symbol TL431
- added D?: LED, symbol LED
- added P?: CONN_01X02, symbol CONN_01X02
- added P? (x6): CONN_01X01, symbol CONN_01X01
- added P? (x3): CONN_01X03, Pin_Headers:Pin_Header_Straight_1x03_Pitch2.54mm, symbol CONN_01X03
- added P? (x2): CONN_01X01, Pin_Headers:Pin_Header_Straight_1x01_Pitch2.54mm, symbol CONN_01X01
- added P? (x2): CONN_01X02, Pin_Headers:Pin_Header_Straight_1x02_Pitch2.54mm, symbol CONN_01X02
- added P?: CONN_02X02, symbol CONN_02X02
- added Q?: BC547, TO-92, symbol BC547
- added Q?: Q_PNP_BCE, symbol Q_PNP_BCE
- added R?: 15.8k, symbol R
- added R? (x9): R, symbol R
- added RV? (x3): POT, symbol POT
- added U?: 7660, symbol 7660
- added U?: OPA547, symbol OPA547-RESCUE-temp_reg
Connections:
- net labels added: +48V, +5V, ADC_CS, ADC_LATCH, DISP_CS, DISP_LATCH, LED_CS, LED_LATCH, stat
- net labels removed: BEEP, CS1, CS2, CS_ADC_A, CS_ADC_B, D4, D5, D6, D7, E, ESTOP, JP_1, JP_2, JP_3, LED_1, LED_2, PWM, PWM_ON/OFF, RW, Vref, a1, a2, a3, segm_a, segm_b, segm_c, segm_d, segm_dp, segm_e, segm_f, segm_g, sw_1, sw_2, sw_3
- wire segments 369 -> 297
- no-connect marks 5 -> 2
Other:
- note added: "beeper-led"
- note added: "displ"
- note removed: "beeper"
- note removed: "comp interface"
- moved on the sheet: 100n?, 10k1, 47u?, P6, R?

Commit message: circuit built
Parts:
- removed 100n? (x4), C1, C2: C_Small, Capacitors_THT:C_Disc_D3.0mm_W1.6mm_P2.50mm, symbol C_Small
- removed 10k1, 220R1, 220R2, 220R4, R1, R10, R2, R22, R23, R6, R7, R9: R, Resistors_THT:Resistor_Horizontal_RM7mm, symbol R
- removed 47u2, 47u3, 47u? (x4): CP1_Small, Capacitors_THT:CP_Radial_D4.0mm_P1.50mm, symbol CP1_Small
- removed C? (x2): CP, symbol CP
- removed E1: Encoder_switch, Pin_Headers:Pin_Header_Straight_1x05_Pitch2.54mm, symbol Encoder_switch
- removed P12, P15, P5, P? (x2): CONN_01X02, Pin_Headers:Pin_Header_Straight_1x02_Pitch2.54mm, symbol CONN_01X02
- removed P2, P? (x3): CONN_01X03, Pin_Headers:Pin_Header_Straight_1x03_Pitch2.54mm, symbol CONN_01X03
- removed P6: CONN_01X04, Pin_Headers:Pin_Header_Straight_1x04_Pitch2.54mm, symbol CONN_01X04
- removed P?: CONN_01X02, symbol CONN_01X02
- removed P? (x2): CONN_01X01, symbol CONN_01X01
- removed P? (x2): CONN_01X01, Pin_Headers:Pin_Header_Straight_1x01_Pitch2.54mm, symbol CONN_01X01
- removed Q?: Q_PNP_BCE, symbol Q_PNP_BCE
- removed R28: 1k, Resistors_THT:Resistor_Horizontal_RM7mm, symbol R
- removed R? (x6): R, symbol R
- removed RV?: POT, symbol POT
- removed U5, U7, U9: EL817C, Housings_DIP:DIP-4_W7.62mm, symbol EL817C-RESCUE-temp_reg
- removed U?: MCP4822-E/MS, SOP65P490X110-8N, symbol MCP4822-E/MS
- removed U?: ATTINY2313A-PU, DIP20, symbol ATTINY2313A-PU
- removed U?: LM393, symbol LM393
- removed U?: 7660, symbol 7660
- added C2: CP, Capacitors_THT:CP_Radial_D7.5mm_P2.50mm, symbol CP
- added P10: CONN_01X02, Pin_Headers:Pin_Header_Straight_1x02_Pitch2.54mm, symbol CONN_01X02
- added P11, P8: CONN_2, borniers:bornier2_V, symbol CONN_2
- added P13, P14, P7: CONN_01X01, Mounting_Holes:MountingHole_3.5mm, symbol CONN_01X01
- added P2: CONN_01X01, Pin_Headers:Pin_Header_Straight_1x01_Pitch2.54mm, symbol CONN_01X01
- added R11, R12: R, Resistors_THT:R_Axial_Power_L20.0mm_W6.4mm_P25.40mm, symbol R
- added R14: R, Resistors_THT:R_Axial_DIN0207_L6.3mm_D2.5mm_P10.16mm_Horizontal, symbol R
- added RV3: POT, Potentiometers:Potentiometer_Trimmer_Bourns_PV36W, symbol POT
- 10u1: footprint Capacitors_THT:CP_Radial_D4.0mm_P1.50mm -> Capacitors_THT:CP_Radial_D5.0mm_P2.50mm
- 47u1: renamed from 47u?; footprint Capacitors_THT:CP_Radial_D4.0mm_P1.50mm -> Capacitors_THT:CP_Radial_D5.0mm_P2.50mm
- C1: renamed from C?; footprint (none) -> Capacitors_THT:CP_Radial_D7.5mm_P2.50mm
- D1: renamed from D?; footprint (none) -> LEDs:LED_D3.0mm
- D2: renamed from D?; footprint (none) -> TO_SOT_Packages_THT:TO-92_Inline_Wide
- P1, P12, P3, P6: renamed from P?; footprint (none) -> Pin_Headers:Pin_Header_Straight_1x01_Pitch2.54mm
- P5: renamed from P?; footprint (none) -> Pin_Headers:Pin_Header_Straight_2x02_Pitch2.54mm
- P9: footprint Pin_Headers:Pin_Header_Straight_1x01_Pitch2.54mm -> Mounting_Holes:MountingHole_3.5mm
- Q1: renamed from Q?; footprint TO-92 -> TO_SOT_Packages_THT:TO-92_Inline_Wide
- R1, R10, R2, R3, R4, R5, R7, R8, R9: renamed from R?; footprint (none) -> Resistors_THT:R_Axial_DIN0207_L6.3mm_D2.5mm_P10.16mm_Horizontal
- R6: renamed from R?; footprint (none) -> Resistors_THT:R_Axial_Power_L20.0mm_W6.4mm_P25.40mm
- RV1, RV2: renamed from RV?; footprint (none) -> Potentiometers:Potentiometer_Trimmer_Bourns_PV36W
- U1: renamed from U?; footprint (none) -> TO_SOT_Packages_THT:TO-220-7_Vertical_StaggeredType2; symbol OPA547-RESCUE-temp_reg -> OPA547-RESCUE-temp_reg-RESCUE-temp_reg
- U11: footprint TO_SOT_Packages_THT:TO-220_Vertical -> TO_SOT_Packages_THT:TO-220_Neutral123_Vertical
- U2: renamed from U?; footprint SOIC127P600X175-8N -> Housings_DIP:DIP-8_W7.62mm_LongPads
- gave numbers to parts that had none: 1
Connections:
- net labels added: +8V
- net labels removed: +12V, ADC_CS, ADC_LATCH, AVCC, DISP_CS, DISP_LATCH, GND, GNDA, IN1, LED_CS, LED_LATCH, MISO, MOSI, OUT1, OUT2, OUT3, RST, SCK, VCC, enc_A, enc_B, stat, sw_e
- wire segments 297 -> 106
- no-connect marks 2 -> 0
Other:
- note removed: "beeper-led"
- note removed: "displ"
- note removed: "emergency stop"
- note removed: "manual / auto"
- note removed: "on / off"
- note removed: "on/off wire heating"
- note removed: "prog"
- note removed: "switches"
- note removed: "usbasp"
- moved on the sheet: 100n1, 100n10, 100n11, 10u1, 47u1, C1, D2, P1, P12, P3, P4, P6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

Commit message: changed current sensing method, added lm358, lm7812, icl7660
Parts:
- added C? (x2): CP, symbol CP
- added R? (x5): R, symbol R
- added RV?: POT, symbol POT
- added U?: 7660, symbol 7660
- added U? (x2): LM358, symbol LM358
- added U?: LM7812, symbol LM7812
Changed lines of the file:
@@
 	1    0    0    -1
 $EndComp
+$Comp
+L 7660 U?
+U 1 1 5A2E24FE
+P 12875 5900
+F 0 "U?" H 12475 6250 50  0000 L CNN
+F 1 "7660" H 12475 5550 50  0000 L CNN
+F 2 "" H 12875 5900 50  0001 C CNN
+F 3 "" H 12875 5900 50  0001 C CNN
+	1    12875 5900
+	1    0    0    -1
+$EndComp
+$Comp
+L LM358 U?
+U 1 1 5A2E28A5
+P 15400 4800
+F 0 "U?" H 15400 5000 50  0000 L CNN
+F 1 "LM358" H 15400 4600 50  0000 L CNN
+F 2 "" H 15400 4800 50  0001 C CNN
+F 3 "" H 15400 4800 50  0001 C CNN
+	1    15400 4800
+	1    0    0    -1
+$EndComp
+$Comp
+L LM358 U?
+U 2 1 5A2E2AD0
+P 16575 4800
+F 0 "U?" H 16575 5000 50  0000 L CNN
+F 1 "LM358" H 16575 4600 50  0000 L CNN
+F 2 "" H 16575 4800 50  0001 C CNN
+F 3 "" H 16575 4800 50  0001 C CNN
+	2    16575 4800
+	1    0    0    1
+$EndComp
+$Comp
+L POT RV?
+U 1 1 5A2E2B87
+P 14550 4700
+F 0 "RV?" V 14375 4700 50  0000 C CNN
+F 1 "POT" V 14450 4700 50  0000 C CNN
+F 2 "" H 14550 4700 50  0001 C CNN
+F 3 "" H 14550 4700 50  0001 C CNN
+	1    14550 4700
+	1    0    0    -1
+$EndComp
+$Comp
+L R R?
+U 1 1 5A2E2ECD
+P 14900 4700
+F 0 "R?" V 14980 4700 50  0000 C CNN
+F 1 "R" V 14900 4700 50  0000 C CNN
+F 2 "" V 14830 4700 50  0001 C CNN
+F 3 "" H 14900 4700 50  0001 C CNN
+	1    14900 4700
+	0    1    1    0
+$EndComp
+$Comp
+L R R?
+U 1 1 5A2E2FFB
+P 14900 4400
+F 0 "R?" V 14980 4400 50  0000 C CNN
+F 1 "R" V 14900 4400 50  0000 C CNN
+F 2 "" V 14830 4400 50  0001 C CNN
+F 3 "" H 14900 4400 50  0001 C CNN
+	1    14900 4400
+	0    1    1    0
+$EndComp
+$Comp
+L R R?
+U 1 1 5A2E30DC
+P 15600 4400
+F 0 "R?" V 15680 4400 50  0000 C CNN
+F 1 "R" V 15600 4400 50  0000 C CNN
+F 2 "" V 15530 4400 50  0001 C CNN
+F 3 "" H 15600 4400 50  0001 C CNN
+	1    15600 4400
+	0    1    1    0
+$EndComp
+$Comp
+L R R?
+U 1 1 5A2E3C2F
+P 16775 4400
+F 0 "R?" V 16855 4400 50  0000 C CNN
+F 1 "R" V 16775 4400 50  0000 C CNN
+F 2 "" V 16705 4400 50  0001 C CNN
+F 3 "" H 16775 4400 50  0001 C CNN
+	1    16775 4400
+	0    1    1    0
+$EndComp
+$Comp
+L R R?
+U 1 1 5A2E3D3A
+P 16000 4800
+F 0 "R?" V 16080 4800 50  0000 C CNN
+F 1 "R" V 16000 4800 50  0000 C CNN
+F 2 "" V 15930 4800 50  0001 C CNN
+F 3 "" H 16000 4800 50  0001 C CNN
+	1    16000 4800
+	0    1    1    0
+$EndComp
+$Comp
+L LM7812 U?
+U 1 1 5A2E3E46
+P 11450 4825
+F 0 "U?" H 11600 4629 50  0000 C CNN
+F 1 "LM7812" H 11450 5025 50  0000 C CNN
+F 2 "" H 11450 4825 50  0001 C CNN
+F 3 "" H 11450 4825 50  0001 C CNN
+	1    11450 4825
+	1    0    0    -1
+$EndComp
+$Comp
+L CP C?
+U 1 1 5A2E403D
+P 12025 6050
+F 0 "C?" H 12050 6150 50  0000 L CNN
+F 1 "CP" H 12050 5950 50  0000 L CNN
+F 2 "" H 12063 5900 50  0001 C CNN
+F 3 "" H 12025 6050 50  0001 C CNN
+	1    12025 6050
+	1    0    0    -1
+$EndComp
+$Comp
+L CP C?
+U 1 1 5A2E4190
+P 13675 6275
+F 0 "C?" H 13700 6375 50  0000 L CNN
+F 1 "CP" H 13700 6175 50  0000 L CNN
+F 2 "" H 13713 6125 50  0001 C CNN
+F 3 "" H 13675 6275 50  0001 C CNN
+	1    13675 6275
+	-1   0    0    1
+$EndComp
 $EndSCHEMATC

Commit message: 1
Parts:
- removed C? (x2): CP, symbol CP
- removed D1: LED, LEDs:LED_D3.0mm, symbol LED
- removed D2: TL431, TO_SOT_Packages_THT:TO-92_Inline_Wide, symbol TL431
- removed P1, P12, P2, P3, P6: CONN_01X01, Pin_Headers:Pin_Header_Straight_1x01_Pitch2.54mm, symbol CONN_01X01
- removed P10: CONN_01X02, Pin_Headers:Pin_Header_Straight_1x02_Pitch2.54mm, symbol CONN_01X02
- removed P4: CONN_2, borniers:bornier2_V, symbol CONN_2
- removed P5: CONN_02X02, Pin_Headers:Pin_Header_Straight_2x02_Pitch2.54mm, symbol CONN_02X02
- removed Q1: BC547, TO_SOT_Packages_THT:TO-92_Inline_Wide, symbol BC547
- removed R10, R14, R3, R5, R7: R, Resistors_THT:R_Axial_DIN0207_L6.3mm_D2.5mm_P10.16mm_Horizontal, symbol R
- removed R? (x5): R, symbol R
- removed RV1, RV3: POT, Potentiometers:Potentiometer_Trimmer_Bourns_PV36W, symbol POT
- removed RV?: POT, symbol POT
- removed U11: LM7805, TO_SOT_Packages_THT:TO-220_Neutral123_Vertical, symbol LM7805-RESCUE-temp_reg
- removed U2: max4210, Housings_DIP:DIP-8_W7.62mm_LongPads, symbol max4210-RESCUE-temp_reg
- removed U?: 7660, symbol 7660
- removed U? (x2): LM358, symbol LM358
- removed U?: LM7812, symbol LM7812
- added 100n4, 100n5: C_Small, Capacitors_THT:C_Disc_D3.0mm_W1.6mm_P2.50mm, symbol C_Small
- added 20k1: POT, Pin_Headers:Pin_Header_Straight_1x03_Pitch2.54mm, symbol POT
- added 20k2, R4, R9: R, Resistors_THT:R_Axial_DIN0207_L6.3mm_D2.5mm_P10.16mm_Horizontal, symbol R
- added 20k3: POT, Potentiometers:Potentiometer_Trimmer_Bourns_PV36W, symbol POT
- added C3, C4: CP, Capacitors_THT:CP_Radial_D7.5mm_P2.50mm, symbol CP
- added D1: TL431, TO_SOT_Packages_THT:TO-92_Inline_Wide, symbol TL431
- added P1: CONN_01X02, Pin_Headers:Pin_Header_Straight_1x02_Pitch2.54mm, symbol CONN_01X02
- added P2: CONN_01X04, Pin_Headers:Pin_Header_Straight_1x04_Pitch2.54mm, symbol CONN_01X04
- added P3: CONN_2, borniers:bornier2_V, symbol CONN_2
- added R11: 20k, Resistors_THT:R_Axial_DIN0207_L6.3mm_D2.5mm_P10.16mm_Horizontal, symbol R
- added RV2: 490k, Potentiometers:Potentiometer_Trimmer_Bourns_PV36W, symbol POT
- added U2: MCP602, Housings_DIP:DIP-8_W7.62mm_Socket_LongPads, symbol MCP602
- added U3: PC817, DIP-4, symbol PC817
- added U4: lt2940, Housings_DIP:DIP-12_W8.89mm_SMDSocket_LongPads, symbol lt2940
- added U5: LM7812, TO_SOT_Packages_THT:TO-220-3_Vertical, symbol LM7812
- added U6: LM7805, TO_SOT_Packages_THT:TO-220-3_Vertical, symbol LM7805
- R2: value R -> 20k
- R3: renamed from R4; value 15.8k -> 200k
- renumbered 100n10 to 100n2, 100n11 to 100n3, C2 to C1, C1 to C2, P8 to P11, P11 to P13, P7 to P6, P9 to P7, P13 to P8, P14 to P9, R9 to R10, R6 to R5, R11 to R6, R12 to R7, RV2 to RV1
Connections:
- net labels added: +12V, Vref, imon, pmon, tmon
- net labels removed: +8V
- wire segments 106 -> 132
- no-connect marks 0 -> 3
Other:
- moved on the sheet: 100n1, 100n2, 100n3, 47u1, C1, C2, P11, P13, P6, P7, P8, P9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

Commit message: working version
Parts:
- removed 100n1, 100n2, 100n3, 100n4, 100n5: C_Small, Capacitors_THT:C_Disc_D3.0mm_W1.6mm_P2.50mm, symbol C_Small
- removed 10u1, 47u1: CP1_Small, Capacitors_THT:CP_Radial_D5.0mm_P2.50mm, symbol CP1_Small
- removed 20k1: POT, Pin_Headers:Pin_Header_Straight_1x03_Pitch2.54mm, symbol POT
- removed 20k2, R1, R10, R4, R8, R9: R, Resistors_THT:R_Axial_DIN0207_L6.3mm_D2.5mm_P10.16mm_Horizontal, symbol R
- removed 20k3, RV1: POT, Potentiometers:Potentiometer_Trimmer_Bourns_PV36W, symbol POT
- removed C2, C3, C4: CP, Capacitors_THT:CP_Radial_D7.5mm_P2.50mm, symbol CP
- removed D1: TL431, TO_SOT_Packages_THT:TO-92_Inline_Wide, symbol TL431
- removed P1: CONN_01X02, Pin_Headers:Pin_Header_Straight_1x02_Pitch2.54mm, symbol CONN_01X02
- removed P13, P3: CONN_2, borniers:bornier2_V, symbol CONN_2
- removed P2: CONN_01X04, Pin_Headers:Pin_Header_Straight_1x04_Pitch2.54mm, symbol CONN_01X04
- removed P6, P7, P8, P9: CONN_01X01, Mounting_Holes:MountingHole_3.5mm, symbol CONN_01X01
- removed R11, R2: 20k, Resistors_THT:R_Axial_DIN0207_L6.3mm_D2.5mm_P10.16mm_Horizontal, symbol R
- removed R3: 200k, Resistors_THT:R_Axial_DIN0207_L6.3mm_D2.5mm_P10.16mm_Horizontal, symbol R
- removed R5, R6, R7: R, Resistors_THT:R_Axial_Power_L20.0mm_W6.4mm_P25.40mm, symbol R
- removed RV2: 490k, Potentiometers:Potentiometer_Trimmer_Bourns_PV36W, symbol POT
- removed U1: OPA547, TO_SOT_Packages_THT:TO-220-7_Vertical_StaggeredType2, symbol OPA547-RESCUE-temp_reg-RESCUE-temp_reg
- removed U2: MCP602, Housings_DIP:DIP-8_W7.62mm_Socket_LongPads, symbol MCP602
- removed U3: PC817, DIP-4, symbol PC817
- removed U4: lt2940, Housings_DIP:DIP-12_W8.89mm_SMDSocket_LongPads, symbol lt2940
- removed U5: LM7812, TO_SOT_Packages_THT:TO-220-3_Vertical, symbol LM7812
- removed U6: LM7805, TO_SOT_Packages_THT:TO-220-3_Vertical, symbol LM7805
- added 1000uF1, C3: CP, Capacitors_THT:CP_Radial_D25.0mm_P10.00mm_SnapIn, symbol device:CP
- added 100n1: C_Small, Capacitors_THT:C_Disc_D3.0mm_W1.6mm_P2.50mm, symbol device:C_Small
- added 10u1, 10u2, 10u3, 10u4: CP1_Small, Capacitors_THT:CP_Radial_D5.0mm_P2.50mm, symbol device:CP1_Small
- added 20k1, R1, R10, R11, R12, R13, R14, R2, R220, R3, R4, R5, R6, R7, R8, R9: R, Resistors_THT:R_Axial_DIN0207_L6.3mm_D2.5mm_P10.16mm_Horizontal, symbol device:R
- added C4: CP, Capacitors_THT:CP_Radial_D7.5mm_P2.50mm, symbol device:CP
- added C5, C7, C8: C_Small, Capacitors_THT:C_Disc_D4.3mm_W1.9mm_P5.00mm, symbol device:C_Small
- added C6: C_Small, Resistors_THT:R_Axial_DIN0207_L6.3mm_D2.5mm_P10.16mm_Horizontal, symbol device:C_Small
- added D1, D2: SCHOTTKY, Diodes_ThroughHole:D_A-405_P12.70mm_Horizontal, symbol w_device:SCHOTTKY
- added D3: LED, LEDs:LED_D4.0mm, symbol device:LED
- added H1, H2, H3, H4: MountingHole, Mounting_Holes:MountingHole_3.2mm_M3, symbol Mechanical:MountingHole
- added L1: L, Inductors_THT:L_Axial_L5.3mm_D2.2mm_P7.62mm_Horizontal_Vishay_IM-1, symbol device:L
- added L2: toroid, Inductors_THT:L_Toroid_Vertical_L21.6mm_W9.5mm_P7.11mm_Pulse_C, symbol device:L
- added P1, P7: CONN_01X03, Pin_Headers:Pin_Header_Straight_1x03_Pitch2.54mm, symbol conn:CONN_01X03
- added P10, P2, P3, P5: CONN_01X01, Pin_Headers:Pin_Header_Straight_1x01_Pitch2.54mm, symbol conn:CONN_01X01
- added P4: CONN_2, borniers:bornier2_V, symbol borniers:CONN_2
- added P6: CONN_01X02, Pin_Headers:Pin_Header_Straight_1x02_Pitch2.54mm, symbol conn:CONN_01X02
- added Q1: IRF9540N, TO_SOT_Packages_THT:TO-220-3_Vertical, symbol Transistor_FET:IRF9540N
- added Q2, Q3, Q6: BC547, TO_SOT_Packages_THT:TO-92_Inline_Wide, symbol Transistor_BJT:BC547
- added Q4, Q5, Q8, Q9: BC557, TO_SOT_Packages_THT:TO-92_Inline_Wide, symbol Transistor_BJT:BC557
- added Q7: IRF540N, TO_SOT_Packages_THT:TO-220-3_Vertical, symbol Transistor_FET:IRF540N
- added R15, R16: 0, Resistors_THT:R_Axial_DIN0207_L6.3mm_D2.5mm_P10.16mm_Horizontal, symbol device:R
- added U1: ATTINY84A-PU, Housings_DIP:DIP-14_W7.62mm_Socket_LongPads, symbol atmel:ATTINY84A-PU
- added U2, U4: PC817, Housings_DIP:DIP-4_W7.62mm_LongPads, symbol opto:PC817
- added U3: BUZZER, Buzzers_Beepers:Buzzer_12x9.5RM7.6, symbol buzzer:BUZZER
- C1: footprint Capacitors_THT:CP_Radial_D7.5mm_P2.50mm -> Capacitors_THT:CP_Radial_D10.0mm_P5.00mm; symbol CP -> device:CP
- P11: symbol CONN_2 -> borniers:CONN_2
Connections:
- net +48V: now also C3.1, C4.1, P2.1 (P1), Q1.3 (S), Q2.1 (C), Q5.3 (E), Q6.1 (C), R1.1
- net +5V: now also 100n1.1, 10u2.1, 10u3.1, 10u4.1, 20k1.1, D3.2 (A), L1.1, P1.1 (P1), Q8.3 (E), R8.1, U1.1 (VCC)
- net GNDPWR: now also 1000uF1.2, C3.2, C4.2, D2.1 (A), P10.1 (P1), Q7.3 (S), R16.2, R4.2, R5.2
- new net: 20k1.2, U1.4 ((PCINT11/dW/~RESET~)PB3)
- new net: Q1.1 (G), Q2.3 (E), Q4.3 (E)
- new net: D2.2 (K), L2.2, Q1.2 (D)
- new net: Q6.3 (E), Q7.1 (G), Q9.3 (E)
- new net: D1.1 (A), L2.1, Q7.2 (D)
- new net: C5.1, Q2.2 (B), Q4.2 (B), R3.1
- new net: Q3.3 (E), Q4.1 (C), Q9.1 (C), R12.2, R16.1
- new net: Q8.1 (C), U3.1 (VCC)
- new net: D3.1 (K), R220.1
- new net: C5.2, Q3.1 (C), R1.2, R3.2
- new net: C6.1, Q3.2 (B), R6.1
- new net: C8.1, Q6.2 (B), Q9.2 (B), R9.1
- new net: 1000uF1.1, D1.2 (K), P4.1 (P1), R2.1
- new net: C8.2, Q5.1 (C), R12.1, R9.2
- new net: C7.1, Q5.2 (B), R7.1
- new net: P7.1 (P1), U4.3
- new net: P7.2 (P2), R14.1
- new net: P7.3 (P3), R14.2, U4.4
- new net: P6.1 (P1), R10.2
- new net: P6.2 (P2), U2.2
- new net: P4.2 (P2), R15.2, R5.1
- new net: R10.1, U2.1
- new net: R13.2, U4.1
- new net: Q8.2 (B), R11.1
- new net: 10u1.1, L1.2, P3.1 (P1)
- new net GND: 100n1.2, 10u1.2, 10u2.2, 10u3.2, 10u4.2, P1.3 (P3), P5.1 (P1), U1.14 (GND), U2.3, U3.2 (GND), U4.2
- new net adc_in: P1.2 (P2), U1.10 ((PCINT3/T0/ADC3)PA3)
- new net beep: R11.2, U1.9 ((PCINT4/USCK/SCL/T1/ADC4)PA4)
- new net i1: C6.2, R6.2, U1.8 ((PCINT5/DO/MISO/OC1B/ADC5)PA5)
- new net i2: C7.2, R7.2, U1.7 ((PCINT6/SDA/DI/MOSI/OC1A/ADC6)PA6)
- new net led: R220.2, U1.3 ((PCINT9/XTAL2)PB1)
- new net oi: R15.1, U1.11 ((PCINT2/AIN1/ADC2)PA2)
- new net ov: R2.2, R4.1, U1.12 ((PCINT1/AIN0/ADC1)PA1)
- new net pwm_in: R8.2, U1.6 ((PCINT7/ICP/OC0B/ADC7)PA7), U2.4
- new net sig_out: R13.1, U1.2 ((PCINT8/CLKI/XTAL1)PB0)
- no-connect marks 3 -> 0
Other:
- moved on the sheet: C1, P11
