File: _saved_temp_reg.sch (KiCad schematic (older format))
At the start: 125 parts

Commit message: start reducing number of components
Parts:
- added D? (x3): Led_Small, symbol Led_Small
- added R? (x3): R, symbol R
Connections:
- net +5V: now also R?.1, R?.1, R?.1
- net OUT1: now also D?.1 (K)
- net OUT2: now also D?.1 (K)
- net OUT3: now also D?.1 (K)
- new net: D?.2 (A), R?.2 (x3)
Other:
- note added: "on / off"
- note added: "prog"
- moved on the sheet: C?, JP?, P?, R?, U?
