File: temp_reg.kicad_pcb (KiCad board)
At the start: 2 copper layers, 262.4 x 161.4 mm, 121 parts, among them IC1 ATMEGA644-P, P1 CONN_01X02, P10 CONN_01X04, P11 CONN_01X06, P12 CONN_01X02, P13 CONN_01X02, P14 CONN_2vert, P15 CONN_01X02, P2 CONN_01X03, P3 CONN_01X03, P4 CONN_2, P5 CONN_01X02, P6 CONN_01X04, P7 CONN_01X06, P8 CONN_01X05, P9 CONN_01X01, Q1 Q_NMOS_DSG, Q2 Q_NMOS_DSG, U1 MCP601P, U10 LM7805, U11 LM7805, U2 MCP3201-CI/SN, U3 MCP601P, U4 MCP3201-CI/SN, U5 EL817C, U6 LM393, U7 EL817C, U8 EL817C, U9 EL817C

Commit message: circuit built
Parts:
- removed 100n2, 100n3, 100n4, 100n5, 100n6, 100n7, 100n8, 100n9, 22p1, 22p2, C7, C8: C_Small, Capacitors_THT:C_Disc_D3.0mm_W1.6mm_P2.50mm
- removed 10k1, 1R1, 1R2, 220R1, 220R2, 220R3, 220R4, R13, R15, R16, R17, R18, R19, R20, R21, R22, R23, R24, R25, R26, R27, R29, R30, R31, R32: R, Resistors_THT:Resistor_Horizontal_RM7mm
- removed 20MHz1: Crystal, Crystals:Resonator-2pin_w7.0mm_h2.5mm
- removed 4.7u1, 4.7u2, 4.7u3, 4.7u4, 47u2, 47u3, 47u4, 47u5, 47u6: CP1_Small, Capacitors_THT:CP_Radial_D4.0mm_P1.50mm
- removed C3, C4: CP, Capacitors_THT:C_Radial_D10_L13_P5
- removed C5, C6, C9: CP1_Small, Capacitors_THT:C_Radial_D5_L6_P2.5
- removed D3, D4: D_Schottky_Small, Diodes_THT:Diode_DO-41_SOD81_Horizontal_RM10
- removed D5: TL431, TO_SOT_Packages_THT:TO-92_Inline_Narrow_Oval
- removed E1: Encoder_switch, Pin_Headers:Pin_Header_Straight_1x05_Pitch2.54mm
- removed IC1: ATMEGA644-P, Housings_DIP:DIP-40_W25.4mm_Socket_LongPads
- removed JP1, JP2, JP3, JP4: Jumper_NO_Small, Buttons_Switches_THT:SW_PUSH_6mm_h4.3mm
- removed L1, L2, L3, L4, L5, L6, L7: L, Resistors_THT:Resistor_Horizontal_RM7mm
- removed P15: CONN_01X02, Pin_Headers:Pin_Header_Straight_1x02_Pitch2.54mm
- removed Q2: Q_NMOS_DSG, TO_SOT_Packages_THT:TO-220_Vertical
- removed R28: 1k, Resistors_THT:Resistor_Horizontal_RM7mm
- removed U10: LM7805, TO_SOT_Packages_THT:TO-220_Vertical
- removed U3: MCP601P, Housings_DIP:DIP-8_W7.62mm
- removed U4: MCP3201-CI/SN, Housings_SOIC:SOIC-8_3.9x4.9mm_Pitch1.27mm
- removed U5, U7, U8, U9: EL817C, Housings_DIP:DIP-4_W7.62mm
- removed U6: LM393, Housings_DIP:DIP-8_W7.62mm
- added RV3: POT, Potentiometers:Potentiometer_Trimmer_Bourns_PV36W, F.Cu at (71.8, 26.0)
- 10u1, 47u1: footprint Capacitors_THT:CP_Radial_D4.0mm_P1.50mm -> Capacitors_THT:CP_Radial_D5.0mm_P2.50mm
- C1, C2: value C_Small -> CP; footprint Capacitors_THT:C_Disc_D3.0mm_W1.6mm_P2.50mm -> Capacitors_THT:CP_Radial_D7.5mm_P2.50mm
- D1: value Led_Small -> LED
- D2: value Led_Small -> TL431; footprint LEDs:LED_D3.0mm -> TO_SOT_Packages_THT:TO-92_Inline_Wide
- P1, P12: value CONN_01X02 -> CONN_01X01; footprint Pin_Headers:Pin_Header_Straight_1x02_Pitch2.54mm -> Pin_Headers:Pin_Header_Straight_1x01_Pitch2.54mm
- P10: value CONN_01X04 -> CONN_01X02; footprint Pin_Headers:Pin_Header_Straight_1x04_Pitch2.54mm -> Pin_Headers:Pin_Header_Straight_1x02_Pitch2.54mm
- P11: value CONN_01X06 -> CONN_2; footprint Pin_Headers:Pin_Header_Straight_1x06_Pitch2.54mm -> borniers:bornier2_V
- P13: value CONN_01X02 -> CONN_01X01; footprint Pin_Headers:Pin_Header_Straight_1x02_Pitch2.54mm -> Mounting_Holes:MountingHole_3.5mm
- P14: value CONN_2vert -> CONN_01X01; footprint borniers:bornier2_V -> Mounting_Holes:MountingHole_3.5mm
- P2, P3: value CONN_01X03 -> CONN_01X01; footprint Pin_Headers:Pin_Header_Straight_1x03_Pitch2.54mm -> Pin_Headers:Pin_Header_Straight_1x01_Pitch2.54mm
- P5: value CONN_01X02 -> CONN_02X02; footprint Pin_Headers:Pin_Header_Straight_1x02_Pitch2.54mm -> Pin_Headers:Pin_Header_Straight_2x02_Pitch2.54mm
- P6: value CONN_01X04 -> CONN_01X01; footprint Pin_Headers:Pin_Header_Straight_1x04_Pitch2.54mm -> Pin_Headers:Pin_Header_Straight_1x01_Pitch2.54mm
- P7: value CONN_01X06 -> CONN_01X01; footprint Pin_Headers:Pin_Header_Straight_1x06_Pitch2.54mm -> Mounting_Holes:MountingHole_3.5mm
- P8: value CONN_01X05 -> CONN_2; footprint Pin_Headers:Pin_Header_Straight_1x05_Pitch2.54mm -> borniers:bornier2_V
- P9: footprint Pin_Headers:Pin_Header_Straight_1x01_Pitch2.54mm -> Mounting_Holes:MountingHole_3.5mm
- Q1: value Q_NMOS_DSG -> BC547; footprint TO_SOT_Packages_THT:TO-220_Vertical -> TO_SOT_Packages_THT:TO-92_Inline_Wide
- R1, R10, R14, R2, R3, R5, R7, R8, R9: footprint Resistors_THT:Resistor_Horizontal_RM7mm -> Resistors_THT:R_Axial_DIN0207_L6.3mm_D2.5mm_P10.16mm_Horizontal
- R11, R12, R6: footprint Resistors_THT:Resistor_Horizontal_RM7mm -> Resistors_THT:R_Axial_Power_L20.0mm_W6.4mm_P25.40mm
- R4: value R -> 15.8k; footprint Resistors_THT:Resistor_Horizontal_RM7mm -> Resistors_THT:R_Axial_DIN0207_L6.3mm_D2.5mm_P10.16mm_Horizontal
- RV1, RV2: footprint Potentiometers:Potentiometer_Trimmer_Bourns_3296W -> Potentiometers:Potentiometer_Trimmer_Bourns_PV36W
- U1: value MCP601P -> OPA547; footprint Housings_DIP:DIP-8_W7.62mm -> TO_SOT_Packages_THT:TO-220-7_Vertical_StaggeredType2
- U11: footprint TO_SOT_Packages_THT:TO-220_Vertical -> TO_SOT_Packages_THT:TO-220_Neutral123_Vertical
- U2: value MCP3201-CI/SN -> max4210; footprint Housings_SOIC:SOIC-8_3.9x4.9mm_Pitch1.27mm -> Housings_DIP:DIP-8_W7.62mm_LongPads
- moved Q1 251.1 mm to (33.0, 22.2), turned to 90 degrees
- moved P5 218.2 mm to (47.0, 22.2), turned to 90 degrees
- moved U1 208.1 mm to (22.2, 45.1), turned to 90 degrees
- moved P4 205.1 mm to (82.5, 36.8), turned to 270 degrees
- moved RV2 195.9 mm to (59.1, 41.9)
- moved P14 194.0 mm to (83.8, 18.4)
- moved 100n11 190.1 mm to (77.5, 62.2), turned to 90 degrees
- moved RV1 184.5 mm to (59.7, 21.0), turned to 180 degrees
- moved P7 182.9 mm to (19.1, 18.4), turned to 0 degrees
- moved U11 182.6 mm to (80.6, 59.7), turned to 270 degrees
- moved 47u1 181.0 mm to (71.1, 38.7), turned to 180 degrees
- moved 100n10 176.4 mm to (80.6, 52.7), turned to 0 degrees
- moved U2 166.1 mm to (71.1, 53.3), turned to 180 degrees
- moved 10u1 162.5 mm to (69.2, 34.3), turned to 45 degrees
- moved R4 158.1 mm to (22.2, 48.9), turned to 270 degrees
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Connections:
- 100n1 pad 1: Net-(100n1-Pad1) -> +5V
- 100n1 pad 2: Net-(100n1-Pad2) -> GNDPWR
- 100n10 pad 1: Net-(100n10-Pad1) -> +8V
- 100n10 pad 2: GNDA -> GNDPWR
- 100n11 pad 1: AVCC -> +5V
- 100n11 pad 2: GNDA -> GNDPWR
- 10u1 pad 1: Net-(100n10-Pad1) -> +5V
- 10u1 pad 2: GNDA -> GNDPWR
- 47u1 pad 1: +12V -> +5V
- C1 pad 1: Net-(C1-Pad1) -> +8V
- C1 pad 2: GND -> GNDPWR
- C2 pad 1: Net-(C2-Pad1) -> +48V
- C2 pad 2: GND -> GNDPWR
- D1 pad 1: /LED_1 -> Net-(D1-Pad1)
- D1 pad 2: Net-(D1-Pad2) -> +5V
- D2 pad 1: /LED_2 -> Net-(D2-Pad1)
- D2 pad 2: Net-(D2-Pad2) -> GNDPWR
- P1 pad 1: Net-(IC1-Pad14) -> Net-(P1-Pad1)
- P10 pad 1: (no net) -> GNDPWR
- P10 pad 2: (no net) -> +8V
- P11 pad 1: /D4 -> GNDPWR
- P11 pad 2: /D5 -> Net-(P11-Pad2)
- P12 pad 1: Net-(220R2-Pad2) -> Net-(P12-Pad1)
- P13 pad 1: Net-(P13-Pad1) -> (no net)
- P14 pad 1: GNDPWR -> (no net)
- P2 pad 1: /SCK -> Net-(P2-Pad1)
- P3 pad 1: /BEEP -> Net-(P3-Pad1)
- P4 pad 2: +12V -> +8V
- P5 pad 1: GND -> Net-(P3-Pad1)
- P5 pad 2: AVCC -> Net-(P5-Pad2)
- P6 pad 1: /IN1 -> Net-(P5-Pad2)
- P7 pad 1: GND -> (no net)
- P8 pad 1: GND -> GNDPWR
- P8 pad 2: /ESTOP -> +48V
- P9 pad 1: /RST -> (no net)
- Q1 pad 1: Net-(100n8-Pad1) -> Net-(Q1-Pad1)
- Q1 pad 2: Net-(L1-Pad1) -> Net-(Q1-Pad2)
- Q1 pad 3: Net-(Q1-Pad3) -> GNDPWR
- R1 pad 1: Net-(C1-Pad1) -> Net-(Q1-Pad2)
- R1 pad 2: AVCC -> Net-(P2-Pad1)
- R10 pad 1: /enc_B -> GNDPWR
- R10 pad 2: Net-(C2-Pad1) -> Net-(P12-Pad1)
- R11 pad 1: Net-(100n1-Pad1) -> Net-(R11-Pad1)
- R12 pad 1: GNDA -> Net-(P11-Pad2)
- R14 pad 1: Net-(100n4-Pad2) -> GNDPWR
- R14 pad 2: Net-(R13-Pad1) -> Net-(D2-Pad3)
- R2 pad 1: Net-(C2-Pad1) -> Net-(D2-Pad1)
- R2 pad 2: AVCC -> +5V
- R3 pad 1: Net-(R3-Pad1) -> Net-(Q1-Pad1)
- R3 pad 2: /mes_A -> Net-(D1-Pad1)
- R4 pad 1: Net-(100n1-Pad2) -> Net-(R4-Pad1)
- R4 pad 2: Net-(R3-Pad1) -> GNDPWR
- R5 pad 1: Net-(100n2-Pad1) -> Net-(R5-Pad1)
- R5 pad 2: Net-(100n1-Pad2) -> Net-(R5-Pad2)
- R6 pad 1: Net-(C1-Pad1) -> Net-(R11-Pad1)
- R6 pad 2: Net-(E1-Pad1) -> Net-(R5-Pad2)
- R7 pad 1: /enc_A -> Net-(R7-Pad1)
- R7 pad 2: Net-(C1-Pad1) -> Net-(P11-Pad2)
- R8 pad 1: GND -> GNDPWR
- R8 pad 2: Net-(R3-Pad1) -> Net-(R7-Pad1)
- R9 pad 1: Net-(C2-Pad1) -> Net-(P12-Pad1)
- R9 pad 2: Net-(E1-Pad3) -> Net-(P11-Pad2)
- RV1 pad 1: GNDA -> Net-(D2-Pad1)
- RV1 pad 2: Net-(D5-Pad3) -> Net-(P5-Pad3)
- RV1 pad 3: Vref -> GNDPWR
- RV2 pad 1: VCC -> Net-(R5-Pad1)
- RV2 pad 2: Net-(P7-Pad3) -> Net-(RV2-Pad2)
- RV2 pad 3: GND -> GNDPWR
- U1 pad 1: (no net) -> Net-(P5-Pad2)
- U1 pad 2: Net-(R11-Pad2) -> Net-(P1-Pad1)
- U1 pad 3: Net-(100n2-Pad1) -> Net-(R4-Pad1)
- U1 pad 4: GNDA -> GNDPWR
- U1 pad 5: (no net) -> +48V
- U1 pad 6: Net-(100n1-Pad1) -> Net-(R5-Pad2)
- U1 pad 7: AVCC -> Net-(P2-Pad1)
- U11 pad 1: Net-(100n10-Pad1) -> +8V
- U11 pad 2: GNDA -> GNDPWR
- U11 pad 3: AVCC -> +5V
- U2 pad 1: Vref -> GNDPWR
- U2 pad 2: Net-(100n1-Pad1) -> Net-(P12-Pad1)
- U2 pad 3: GNDA -> (no net)
- U2 pad 4: GNDA -> +5V
- U2 pad 5: /CS_ADC_A -> Net-(RV2-Pad2)
- U2 pad 6: /MOSI -> (no net)
- U2 pad 7: /SCK -> Net-(R7-Pad1)
- U2 pad 8: AVCC -> Net-(P1-Pad1)
Routing:
- net GNDPWR: track 0.00 -> 280.2 mm
- net +5V: track 0.00 -> 75.5 mm
- net Net-(P1-Pad1): track 0.00 -> 49.9 mm, vias 0 -> 2
- net Net-(P5-Pad2): track 0.00 -> 44.2 mm
- net +48V: track 0.00 -> 41.6 mm
- net GND: track 38.6 -> 0.00 mm
- net Net-(R5-Pad2): track 0.00 -> 34.8 mm
- net GNDA: track 31.0 -> 0.00 mm
- net Net-(D2-Pad1): track 0.00 -> 30.6 mm
- net Net-(P2-Pad1): track 0.00 -> 27.2 mm
- net Net-(P11-Pad2): track 0.00 -> 26.7 mm
- net +8V: track 0.00 -> 23.7 mm
- net Net-(C5-Pad1): track 22.0 -> 0.00 mm
- net Net-(P12-Pad1): track 0.00 -> 20.7 mm
- net /BEEP: track 20.7 -> 0.00 mm
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Other:
- board size 262.4 x 161.4 mm -> 72.4 x 57.1 mm

Commit message: 1
Parts:
- added R13: R, Resistors_THT:R_Axial_DIN0207_L6.3mm_D2.5mm_P10.16mm_Horizontal, F.Cu at (121.3, 105.4)
- added U3: max4210, Housings_DIP:DIP-8_W7.62mm_LongPads, F.Cu at (128.3, 78.1)
- added U4: lt2940, Housings_DIP:DIP-12_W8.89mm_SMDSocket_LongPads, F.Cu at (132.1, 94.0)
Routing:
- net (no net): track 0.00 -> 170.9 mm, vias 0 -> 2
- net GNDPWR: track 280.2 -> 325.5 mm
- net Net-(R13-Pad2): track 0.00 -> 35.1 mm
- net Net-(U3-Pad5): track 0.00 -> 33.5 mm, vias 0 -> 2
- net Net-(U3-Pad7): track 0.00 -> 33.0 mm
- net Net-(U3-Pad2): track 0.00 -> 23.9 mm
- net Net-(U3-Pad4): track 0.00 -> 9.79 mm

Commit message: working version
Parts:
- removed 100n10, 100n11: C_Small, Capacitors_THT:C_Disc_D3.0mm_W1.6mm_P2.50mm
- removed 47u1: CP1_Small, Capacitors_THT:CP_Radial_D5.0mm_P2.50mm
- removed C2: CP, Capacitors_THT:CP_Radial_D7.5mm_P2.50mm
- removed P12: CONN_01X01, Pin_Headers:Pin_Header_Straight_1x01_Pitch2.54mm
- removed P13, P14, P9: CONN_01X01, Mounting_Holes:MountingHole_3.5mm
- removed P8: CONN_2, borniers:bornier2_V
- removed RV1, RV2, RV3: POT, Potentiometers:Potentiometer_Trimmer_Bourns_PV36W
- removed U11: LM7805, TO_SOT_Packages_THT:TO-220_Neutral123_Vertical
- added 1000uF1: CP, Capacitors_THT:CP_Radial_D25.0mm_P10.00mm_SnapIn, F.Cu at (182.9, 98.4)
- added 10u2: CP1_Small, Capacitors_THT:CP_Radial_D5.0mm_P2.50mm, F.Cu at (114.3, 104.8)
- added 10u3: CP1_Small, Capacitors_THT:CP_Radial_D5.0mm_P2.50mm, F.Cu at (141.0, 116.2)
- added 10u4: CP1_Small, Capacitors_THT:CP_Radial_D5.0mm_P2.50mm, F.Cu at (167.0, 125.1)
- added 20k1: R, Resistors_THT:R_Axial_DIN0207_L6.3mm_D2.5mm_P10.16mm_Horizontal, F.Cu at (167.0, 121.9)
- added C3: CP, Capacitors_THT:CP_Radial_D25.0mm_P10.00mm_SnapIn, F.Cu at (128.3, 72.4)
- added C4: CP, Capacitors_THT:CP_Radial_D7.5mm_P2.50mm, F.Cu at (145.4, 78.1)
- added C5: C_Small, Capacitors_THT:C_Disc_D4.3mm_W1.9mm_P5.00mm, F.Cu at (158.1, 85.1)
- added C6: C_Small, Resistors_THT:R_Axial_DIN0207_L6.3mm_D2.5mm_P10.16mm_Horizontal, F.Cu at (153.0, 97.2)
- added C7: C_Small, Capacitors_THT:C_Disc_D4.3mm_W1.9mm_P5.00mm, F.Cu at (165.7, 101.6)
- added C8: C_Small, Capacitors_THT:C_Disc_D4.3mm_W1.9mm_P5.00mm, F.Cu at (176.5, 90.2)
- added D3: LED, LEDs:LED_D4.0mm, F.Cu at (148.6, 111.1)
- added H1: MountingHole, Mounting_Holes:MountingHole_3.2mm_M3, F.Cu at (204.5, 67.9)
- added H2: MountingHole, Mounting_Holes:MountingHole_3.2mm_M3, F.Cu at (202.6, 126.4)
- added H3: MountingHole, Mounting_Holes:MountingHole_3.2mm_M3, F.Cu at (110.5, 67.9)
- added H4: MountingHole, Mounting_Holes:MountingHole_3.2mm_M3, F.Cu at (110.5, 126.4)
- added L1: L, Inductors_THT:L_Axial_L5.3mm_D2.2mm_P7.62mm_Horizontal_Vishay_IM-1, F.Cu at (108.6, 106.0)
- added L2: toroid, Inductors_THT:L_Toroid_Vertical_L21.6mm_W9.5mm_P7.11mm_Pulse_C, F.Cu at (174.0, 75.6)
- added Q2: BC547, TO_SOT_Packages_THT:TO-92_Inline_Wide, F.Cu at (158.3, 82.2)
- added Q3: BC547, TO_SOT_Packages_THT:TO-92_Inline_Wide, F.Cu at (156.8, 94.0)
- added Q4: BC557, TO_SOT_Packages_THT:TO-92_Inline_Wide, F.Cu at (152.6, 82.2)
- added Q5: BC557, TO_SOT_Packages_THT:TO-92_Inline_Wide, F.Cu at (169.5, 91.4)
- added Q6: BC547, TO_SOT_Packages_THT:TO-92_Inline_Wide, F.Cu at (197.7, 82.5)
- added Q7: IRF540N, TO_SOT_Packages_THT:TO-220-3_Vertical, F.Cu at (192.4, 73.0)
- added Q8: BC557, TO_SOT_Packages_THT:TO-92_Inline_Wide, F.Cu at (146.1, 120.7)
- added Q9: BC557, TO_SOT_Packages_THT:TO-92_Inline_Wide, F.Cu at (192.0, 82.5)
- added R15: 0, Resistors_THT:R_Axial_DIN0207_L6.3mm_D2.5mm_P10.16mm_Horizontal, F.Cu at (189.9, 112.4)
- added R220: R, Resistors_THT:R_Axial_DIN0207_L6.3mm_D2.5mm_P10.16mm_Horizontal, F.Cu at (150.5, 111.8)
- C1: footprint Capacitors_THT:CP_Radial_D7.5mm_P2.50mm -> Capacitors_THT:CP_Radial_D10.0mm_P5.00mm
- D1: value LED -> SCHOTTKY; footprint LEDs:LED_D3.0mm -> Diodes_ThroughHole:D_A-405_P12.70mm_Horizontal
- D2: value TL431 -> SCHOTTKY; footprint TO_SOT_Packages_THT:TO-92_Inline_Wide -> Diodes_ThroughHole:D_A-405_P12.70mm_Horizontal
- P1: value CONN_01X01 -> CONN_01X03; footprint Pin_Headers:Pin_Header_Straight_1x01_Pitch2.54mm -> Pin_Headers:Pin_Header_Straight_1x03_Pitch2.54mm
- P10: value CONN_01X02 -> CONN_01X01; footprint Pin_Headers:Pin_Header_Straight_1x02_Pitch2.54mm -> Pin_Headers:Pin_Header_Straight_1x01_Pitch2.54mm
- P5: value CONN_02X02 -> CONN_01X01; footprint Pin_Headers:Pin_Header_Straight_2x02_Pitch2.54mm -> Pin_Headers:Pin_Header_Straight_1x01_Pitch2.54mm
- P6: value CONN_01X01 -> CONN_01X02; footprint Pin_Headers:Pin_Header_Straight_1x01_Pitch2.54mm -> Pin_Headers:Pin_Header_Straight_1x02_Pitch2.54mm
- P7: value CONN_01X01 -> CONN_01X03; footprint Mounting_Holes:MountingHole_3.5mm -> Pin_Headers:Pin_Header_Straight_1x03_Pitch2.54mm
- Q1: value BC547 -> IRF9540N; footprint TO_SOT_Packages_THT:TO-92_Inline_Wide -> TO_SOT_Packages_THT:TO-220-3_Vertical
- R11, R12, R6: footprint Resistors_THT:R_Axial_Power_L20.0mm_W6.4mm_P25.40mm -> Resistors_THT:R_Axial_DIN0207_L6.3mm_D2.5mm_P10.16mm_Horizontal
- R4: value 15.8k -> R
- U1: value OPA547 -> ATTINY84A-PU; footprint TO_SOT_Packages_THT:TO-220-7_Vertical_StaggeredType2 -> Housings_DIP:DIP-14_W7.62mm_Socket_LongPads
- U2: value max4210 -> PC817; footprint Housings_DIP:DIP-8_W7.62mm_LongPads -> Housings_DIP:DIP-4_W7.62mm_LongPads
- U3: value max4210 -> BUZZER; footprint Housings_DIP:DIP-8_W7.62mm_LongPads -> Buzzers_Beepers:Buzzer_12x9.5RM7.6
- U4: value lt2940 -> PC817; footprint Housings_DIP:DIP-12_W8.89mm_SMDSocket_LongPads -> Housings_DIP:DIP-4_W7.62mm_LongPads
- moved R4 180.4 mm to (189.9, 115.6), turned to 0 degrees
- moved U1 177.4 mm to (186.1, 113.0), turned to 270 degrees
- moved R2 168.5 mm to (200.0, 118.7), turned to 180 degrees
- moved R1 153.0 mm to (160.7, 91.4), turned to 180 degrees
- moved R5 152.2 mm to (203.8, 103.5), turned to 90 degrees
- moved D1 150.8 mm to (187.3, 71.1), turned to 270 degrees
- moved R3 144.9 mm to (160.7, 88.3), turned to 180 degrees
- moved P4 142.7 mm to (193.7, 126.4), turned to 0 degrees
- moved 100n1 141.1 mm to (186.1, 124.5)
- moved P1 136.7 mm to (173.4, 124.5), turned to 90 degrees
- moved P7 135.8 mm to (131.4, 94.6)
- moved Q1 130.3 mm to (153.0, 73.0), turned to 0 degrees
- moved R12 126.3 mm to (172.1, 95.9), turned to 180 degrees
- moved P5 123.5 mm to (123.2, 119.4)
- moved P6 122.3 mm to (131.4, 102.9)
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Connections:
- 100n1 pad 2: GNDPWR -> GND
- 10u1 pad 1: +5V -> Net-(10u1-Pad1)
- 10u1 pad 2: GNDPWR -> GND
- C1 pad 1: +8V -> +48V
- D1 pad 2: +5V -> Net-(1000uF1-Pad1)
- D2 pad 1: Net-(D2-Pad1) -> GNDPWR
- D2 pad 2: GNDPWR -> Net-(D2-Pad2)
- P1 pad 1: Net-(P1-Pad1) -> +5V
- P11 pad 2: Net-(P11-Pad2) -> +48V
- P2 pad 1: Net-(P2-Pad1) -> +48V
- P3 pad 1: Net-(P3-Pad1) -> Net-(10u1-Pad1)
- P4 pad 1: GNDPWR -> Net-(1000uF1-Pad1)
- P4 pad 2: +8V -> Net-(P4-Pad2)
- P5 pad 1: Net-(P3-Pad1) -> GND
- P6 pad 1: Net-(P5-Pad2) -> Net-(P6-Pad1)
- P7 pad 1: (no net) -> Net-(P7-Pad1)
- Q1 pad 2: Net-(Q1-Pad2) -> Net-(D2-Pad2)
- Q1 pad 3: GNDPWR -> +48V
- R1 pad 1: Net-(Q1-Pad2) -> +48V
- R1 pad 2: Net-(P2-Pad1) -> Net-(C5-Pad2)
- R10 pad 1: GNDPWR -> Net-(R10-Pad1)
- R10 pad 2: Net-(P12-Pad1) -> Net-(P6-Pad1)
- R11 pad 1: Net-(R11-Pad1) -> Net-(Q8-Pad2)
- R11 pad 2: Net-(R11-Pad2) -> /beep
- R12 pad 1: Net-(P11-Pad2) -> Net-(C8-Pad2)
- R12 pad 2: Net-(R11-Pad2) -> GNDPWR
- R13 pad 1: GNDPWR -> /sig_out
- R14 pad 1: GNDPWR -> Net-(P7-Pad2)
- R14 pad 2: Net-(D2-Pad3) -> Net-(P7-Pad3)
- R2 pad 1: Net-(D2-Pad1) -> Net-(1000uF1-Pad1)
- R2 pad 2: +5V -> /ov
- R3 pad 1: Net-(Q1-Pad1) -> Net-(C5-Pad1)
- R3 pad 2: Net-(D1-Pad1) -> Net-(C5-Pad2)
- R4 pad 1: Net-(R4-Pad1) -> /ov
- R5 pad 1: Net-(R5-Pad1) -> Net-(P4-Pad2)
- R5 pad 2: Net-(R5-Pad2) -> GNDPWR
- R6 pad 1: Net-(R11-Pad1) -> Net-(C6-Pad1)
- R6 pad 2: Net-(R5-Pad2) -> /i1
- R7 pad 1: Net-(R7-Pad1) -> Net-(C7-Pad1)
- R7 pad 2: Net-(P11-Pad2) -> /i2
- R8 pad 1: GNDPWR -> +5V
- R8 pad 2: Net-(R7-Pad1) -> /pwm_in
- R9 pad 1: Net-(P12-Pad1) -> Net-(C8-Pad1)
- R9 pad 2: Net-(P11-Pad2) -> Net-(C8-Pad2)
- U1 pad 1: Net-(P5-Pad2) -> +5V
- U1 pad 2: Net-(P1-Pad1) -> /sig_out
- U1 pad 3: Net-(R4-Pad1) -> /led
- U1 pad 4: GNDPWR -> Net-(20k1-Pad2)
- U1 pad 5: +48V -> Net-(U1-Pad5)
- U1 pad 6: Net-(R5-Pad2) -> /pwm_in
- U1 pad 7: Net-(P2-Pad1) -> /i2
- U2 pad 1: GNDPWR -> Net-(R10-Pad1)
- U2 pad 2: Net-(P12-Pad1) -> Net-(P6-Pad2)
- U2 pad 3: (no net) -> GND
- U2 pad 4: +5V -> /pwm_in
- U3 pad 1: GNDPWR -> Net-(Q8-Pad1)
- U3 pad 2: Net-(U3-Pad2) -> GND
- U4 pad 1: (no net) -> Net-(R13-Pad2)
- U4 pad 2: (no net) -> GND
- U4 pad 3: GNDPWR -> Net-(P7-Pad1)
- U4 pad 4: Net-(R13-Pad2) -> Net-(P7-Pad3)
Routing:
- net (no net): track 170.9 -> 0.00 mm, vias 2 -> 0
- net GND: track 0.00 -> 155.8 mm, vias 0 -> 2
- net +48V: track 41.6 -> 186.3 mm, vias 0 -> 4
- net +5V: track 75.5 -> 182.0 mm, vias 0 -> 2
- net GNDPWR: track 325.5 -> 259.9 mm
- net Net-(1000uF1-Pad1): track 0.00 -> 59.3 mm
- net Net-(P1-Pad1): track 49.9 -> 0.00 mm, vias 2 -> 0
- net /sig_out: track 0.00 -> 45.5 mm
- net /pwm_in: track 0.00 -> 44.7 mm
- net Net-(P5-Pad2): track 44.2 -> 0.00 mm
- net Net-(R5-Pad2): track 34.8 -> 0.00 mm
- net Net-(U3-Pad5): track 33.5 -> 0.00 mm, vias 2 -> 0
- net Net-(U3-Pad7): track 33.0 -> 0.00 mm
- net Net-(R13-Pad2): track 35.1 -> 3.70 mm
- net Net-(P4-Pad2): track 0.00 -> 31.0 mm
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Other:
- board size 72.4 x 57.1 mm -> 107.9 x 66 mm
- net class thick added: clearance 0.5, trace_width 2, via_dia 0.6, via_drill 0.4
